File: LEDFlasher.kicad_pcb (KiCad board)
At the start: 2 copper layers, 63.5 x 53.3 mm, 17 parts, among them Q1 2N3904, SW1 SW_Push, T1 Transformer_1P_1S, U1 4001

Commit message: v0.3 production
Parts:
- added REF**: WEEE-Logo_4.2x6mm_SilkScreen, Symbol:WEEE-Logo_4.2x6mm_SilkScreen, B.Cu at (151.7, 111.5)
- added REF**: KiCad-Logo2_6mm_SilkScreen, Symbol:KiCad-Logo2_6mm_SilkScreen, F.Cu at (147.1, 110.3)
- added REF**: Symbol_Attention_CopperTop_Small, Symbol:Symbol_Attention_CopperTop_Small, B.Cu at (130.0, 94.2)
- added REF**: Symbol_Attention_CopperTop_Small, Symbol:Symbol_Attention_CopperTop_Small, F.Cu at (130.0, 94.0)
Other:
- board text added: "For Start push 1x only!"
- board text added: "JLCJLCJLCJLC"
- board text added: "LED Flasher v0.3 Design by ZiliziI"
- board text added: "v0.3"
